File: shelly1pm-programmer.kicad_pcb (KiCad board)
At the start: 2 copper layers, 2 parts

Commit message: Initial version
Parts:
- removed the G*** at (30.5, 184.9)
- added J1: Device Connector, Connector_PinHeader_1.27mm:PinHeader_1x07_P1.27mm_Vertical, B.Cu at (153.7, 90.8)
- added J2: Prog. Hdr., Connector_PinSocket_2.54mm:PinSocket_1x06_P2.54mm_Horizontal, F.Cu at (115.1, 88.3)
- added J3: Debug, Connector_PinSocket_2.54mm:PinSocket_1x02_P2.54mm_Vertical, F.Cu at (133.3, 88.3)
- added Q1: UMH3N, Package_TO_SOT_SMD:SOT-363_SC-70-6, F.Cu at (134.0, 95.7)
- added SW1: Reset, Button_Switch_THT:SW_PUSH_6mm, F.Cu at (138.6, 98.5)
- added SW2: Boot, Button_Switch_THT:SW_PUSH_6mm, F.Cu at (123.8, 98.3)
- moved G*** 122.7 mm to (109.5, 95.9)
Routing:
- net +3V3: track 0.00 -> 52.7 mm
- net ~{RESET}: track 0.00 -> 44.2 mm
- net ESP_TX: track 0.00 -> 40.1 mm
- net ESP_RX: track 0.00 -> 38.6 mm, vias 0 -> 2
- net ~{GPIO0}: track 0.00 -> 35.9 mm
- net DTR: track 0.00 -> 22.3 mm
- net RTS: track 0.00 -> 21.5 mm
- net ESP_DBG: track 0.00 -> 21.4 mm
- added copper zone on B.Cu, net GND
Other:
- board outline added: 53.2 x 19.9 mm
- board text added: "3v3"
- board text added: "DBG TX -> RX <- 3v3 RESET GPIO0 GND"
- board text added: "DTR"
- board text added: "GND"
- board text added: "RTS"
- board text added: "RX <"
- board text added: "Shelly 1pm Programmer v1.0 (c) chof 2024"
- board text added: "TX >"
